Commit message: update

File: urdf/amr_mtt.xacro (robot description, xacro)
@@ -2,11 +2,13 @@
 <robot xmlns:xacro="http://www.ros.org/wiki/xacro" name="amr_mtt">
     <!--................................ XACRO CONSTANTS .............................. -->
-    <xacro:property name="chassis_mass" value="60"/>
+    <!-- หุ่นยนต์หนัก 60 kg -->
+    <xacro:property name="chassis_mass" value="135"/>
     <xacro:property name="chassis_length" value="0.9"/>
     <xacro:property name="chassis_width" value="0.64"/>
     <xacro:property name="chassis_height" value="0.2"/>
-    <xacro:property name="traction_wheel_mass" value="1"/>
+    <!-- traction_wheel_mass (มวลของล้อขับเคลื่อน) -->
+    <xacro:property name="traction_wheel_mass" value="4.6"/>
     <xacro:property name="traction_wheel_base" value="0.88"/>
-    <xacro:property name="traction_max_wheel_torque" value="150000"/>
+    <xacro:property name="traction_max_wheel_torque" value="11.4"/>
     <xacro:property name="traction_wheel_friction" value="3.0"/>
     <xacro:property name="trolley_wheel_mass" value="0.1"/>
@@ -16,6 +18,10 @@
     <!-- a small constant -->
     <xacro:property name="eps" value="0.002"/>
+    <!-- การระบุพารามิเตอร์ "รัศมีล้อ" (Wheel Radius) ระบุเส้นผ่านศูนย์กลางภายนอกสุดที่ 160 mm
+    ค่าที่ต้องใช้จริง: รัศมี = 160 mm / 2 = 80 mm = 0.08 m   -->
     <xacro:property name="traction_wheel_radius" value="0.08"/>
-    <xacro:property name="traction_wheel_width" value="0.05"/>
+    <!--การระบุพารามิเตอร์ "ความกว้างล้อ" (Wheel Width) แบบระบุความกว้างรวมของล้อที่ 160 mm -->
+    <xacro:property name="traction_wheel_width" value="0.06"/>
+    <!-- พารามิเตอร์นี้คือระยะห่างระหว่าง "กึ่งกลางล้อซ้าย" ถึง "กึ่งกลางล้อขวา" -->
     <xacro:property name="traction_track_width" value="0.436"/>
     <xacro:property name="two_d_lidar_update_rate" value="30"/>
@@ -44,13 +50,13 @@
     <xacro:include filename="$(find amr_mtt)/urdf/materials.xacro"/>
     <xacro:include filename="$(find amr_mtt)/urdf/macros.xacro"/>
-    <xacro:if value="$(arg sim_gazebo)">
+    <!-- <xacro:if value="$(arg sim_gazebo)">
         <xacro:include filename="$(find amr_mtt)/urdf/gazebo.xacro"/>
-    </xacro:if>
+    </xacro:if> -->
     <xacro:if value="$(arg sim_ign)">
         <xacro:include filename="$(find amr_mtt)/urdf/ign.xacro"/>
     </xacro:if>
-    <xacro:if value="$(arg sim_gz)">
+    <!-- <xacro:if value="$(arg sim_gz)">
         <xacro:include filename="$(find amr_mtt)/urdf/gz.xacro"/>
-    </xacro:if>
+    </xacro:if> -->
     <!-- ................................ BASE LINK .................................. -->
     <link name="base_footprint"/>
@@ -74,11 +80,12 @@
                 <!-- <mesh filename="file://$(find amr_mtt)/meshes/amr_mtt_mesh.dae" scale="1 1 1"/> -->
             </geometry>
-            <material name="">
-                <color rgba="0.772549019607843 0.752941176470588 0.733333333333333 1" />
-            </material>
+            <material name="orange"/>
         </visual>
-        <inertial>
+       <inertial>
+            <origin xyz="0 0 0.1" rpy="0 0 0"/>
             <mass value="${chassis_mass}" />
-            <xacro:box_inertia m="${chassis_mass}" x="${chassis_length}" y="${chassis_width}" z = "${chassis_height}"/>
+            <inertia ixx="5.058" ixy="0" ixz="0"
+                     iyy="9.562" iyz="0"
+                     izz="13.720" />
         </inertial>
     </link>

File: urdf/ign.xacro (robot description, xacro)
@@ -14,8 +14,12 @@
             <left_joint>middle_left_wheel_joint</left_joint>
             <right_joint>middle_right_wheel_joint</right_joint>
-            <wheel_separation>${traction_track_width+traction_wheel_width-0.01}</wheel_separation>
-            <wheel_radius>${traction_wheel_radius+0.01}</wheel_radius>
-            <odom_publish_frequency>30</odom_publish_frequency>
+            <wheel_separation>${traction_track_width}</wheel_separation>
+            <wheel_radius>${traction_wheel_radius}</wheel_radius>
+            <odom_publish_frequency>50</odom_publish_frequency>
             <topic>/cmd_vel</topic>
+            <max_linear_acceleration>0.8</max_linear_acceleration>
+            <max_angular_acceleration>2.0</max_angular_acceleration>
+            <min_linear_acceleration>-0.8</min_linear_acceleration>
+            <min_angular_acceleration>-2.0</min_angular_acceleration>
             <xacro:if value="${odometry_source == 'encoders'}">
                 <odom_topic>$(arg wheel_odom_topic)</odom_topic>
@@ -128,5 +132,5 @@
         <sensor name="imu_sensor" type="imu">
             <always_on>1</always_on>
-            <update_rate>1</update_rate>
+            <update_rate>50</update_rate>
             <ignition_frame_id>imu_frame</ignition_frame_id>
             <visualize>true</visualize>
@@ -175,3 +179,33 @@
         </gazebo>
     </xacro:if>
+    <!-- ........................... MATERIALS ................................... -->
+    <gazebo reference="base_link">
+        <visual>
+            <material>
+                <pbr>
+                    <metal>
+                        <roughness>0.15</roughness>
+                        <metalness>0.8</metalness>
+                    </metal>
+                </pbr>
+                <ambient>0.2 0.2 0.2 1</ambient>
+                <diffuse>0.5 0.5 0.5 1</diffuse>
+                <specular>1 1 1 1</specular>
+            </material>
+        </visual>
+    </gazebo>
+    <gazebo reference="middle_left_wheel">
+        <visual>
+            <material>
+                <pbr>
+                    <metal>
+                        <roughness>0.8</roughness>
+                        <metalness>0.0</metalness>
+                    </metal>
+                </pbr>
+                <ambient>0.1 0.1 0.1 1</ambient>
+                <diffuse>0.1 0.1 0.1 1</diffuse>
+            </material>
+        </visual>
+    </gazebo>
 </robot>

Commit message: ีupdate

File: urdf/amr_mtt.xacro (robot description, xacro)
@@ -77,6 +77,6 @@
             <origin xyz="0 0 0" rpy="0 0 0" />
             <geometry>
-                <mesh filename="file://$(find amr_mtt)/meshes/amr_mtt_model/base_link.STL" scale="1 1 1"/>
-                <!-- <mesh filename="file://$(find amr_mtt)/meshes/amr_mtt_mesh.dae" scale="1 1 1"/> -->
+                <!-- <mesh filename="file://$(find amr_mtt)/meshes/amr_mtt_model/base_link.STL" scale="1 1 1"/> -->
+                <mesh filename="package://amr_mtt/meshes/amr_mtt_model/base_link.STL" scale="1 1 1"/>
             </geometry>
             <material name="orange"/>
@@ -111,16 +111,14 @@
                 <origin xyz="0 0 0" rpy="0 0 0"/>
                 <geometry>
-                    <!-- <mesh filename="package://amr_mtt/meshes/amr_mtt_model/L_F_Lidar_Link.STL" scale="1 1 1"/> -->
-                    <mesh filename="file://$(find amr_mtt)/meshes/amr_mtt_model/L_F_Lidar_Link.STL" scale="1 1 1"/>
-                </geometry>
-            </collision>
-            <visual>
-                <origin xyz="0 0 0" rpy="0 0 0"/>
-                <geometry>
-                    <!-- <mesh filename="package://amr_mtt/meshes/amr_mtt_model/L_F_Lidar_Link.STL" scale="1 1 1"/> -->
-                    <mesh filename="file://$(find amr_mtt)/meshes/amr_mtt_model/L_F_Lidar_Link.STL" scale="1 1 1"/>
-                </geometry>
-                <material name="blue">
-                    <color rgba="0 0 1 1" />
+                   <mesh filename="package://amr_mtt/meshes/amr_mtt_model/L_F_Lidar_Link.STL" scale="1 1 1"/>
+                </geometry>
+            </collision>
+            <visual>
+                <origin xyz="0 0 0" rpy="0 0 0"/>
+                <geometry>
+                    <mesh filename="package://amr_mtt/meshes/amr_mtt_model/L_F_Lidar_Link.STL" scale="1 1 1"/>
+                </geometry>
+                <material name="black">
+                    <color rgba="0 0 0 1" />
                 </material>
             </visual>
@@ -148,15 +146,14 @@
                 <origin xyz="0 0 0" rpy="0 0 0"/>
                 <geometry>
-                    <!-- <mesh filename="package://amr_mtt/meshes/amr_mtt_model/R_B_Lidar_Link.STL" scale="1 1 1"/> -->
-                    <mesh filename="file://$(find amr_mtt)/meshes/amr_mtt_model/R_B_Lidar_Link.STL" scale="1 1 1"/>
-                </geometry>
-            </collision>
-            <visual>
-                <origin xyz="0 0 0" rpy="0 0 0"/>
-                <geometry>
-                    <mesh filename="file://$(find amr_mtt)/meshes/amr_mtt_model/R_B_Lidar_Link.STL" scale="1 1 1"/>
-                </geometry>
-                <material name="blue">
-                    <color rgba="0 0 1 1" />
+                    <mesh filename="package://amr_mtt/meshes/amr_mtt_model/R_B_Lidar_Link.STL" scale="1 1 1"/>
+                </geometry>
+            </collision>
+            <visual>
+                <origin xyz="0 0 0" rpy="0 0 0"/>
+                <geometry>
+                    <mesh filename="package://amr_mtt/meshes/amr_mtt_model/R_B_Lidar_Link.STL" scale="1 1 1"/>
+                </geometry>
+                <material name="black">
+                    <color rgba="0 0 0 1" />
                 </material>
             </visual>
@@ -191,15 +188,14 @@
                 <origin xyz="0 0 0" rpy="0 0 0" />
                 <geometry>
-                    <mesh filename="file://$(find amr_mtt)/meshes/amr_mtt_model/F_Cam_Link.STL" scale="1 1 1"/>
-                </geometry>
-            </collision>
-            <visual>
-                <origin xyz="0 0 0" rpy="0 0 0" />
-                <geometry>
-                    <!-- <mesh filename="file://$(find amr_mtt)/meshes/kinect/d415.dae"/> -->
-                    <mesh filename="file://$(find amr_mtt)/meshes/amr_mtt_model/F_Cam_Link.STL" scale="1 1 1"/>
-                </geometry>
-                <material name="red">
-                    <color rgba="1 0 0 1" />
+                    <mesh filename="package://amr_mtt/meshes/amr_mtt_model/F_Cam_Link.STL" scale="1 1 1"/>
+                </geometry>
+            </collision>
+            <visual>
+                <origin xyz="0 0 0" rpy="0 0 0" />
+                <geometry>
+                    <mesh filename="package://amr_mtt/meshes/amr_mtt_model/F_Cam_Link.STL" scale="1 1 1"/>
+                </geometry>
+                <material name="blue">
+                    <color rgba="0 0 1 1" />
                 </material>
             </visual>
@@ -228,11 +224,11 @@
                 <origin xyz="0 0 0" rpy="0 0 0" />
                 <geometry>
-                    <mesh filename="file://$(find amr_mtt)/meshes/amr_mtt_model/F_Cam_Link.STL" scale="1 1 1"/>
-                </geometry>
-            </collision>
-            <visual>
-                <origin xyz="0 0 0" rpy="0 0 0" />
-                <geometry>
-                    <mesh filename="file://$(find amr_mtt)/meshes/amr_mtt_model/F_Cam_Link.STL" scale="1 1 1"/>
+                    <mesh filename="package://amr_mtt/meshes/amr_mtt_model/F_Cam_Link.STL" scale="1 1 1"/>
+                </geometry>
+            </collision>
+            <visual>
+                <origin xyz="0 0 0" rpy="0 0 0" />
+                <geometry>
+                    <mesh filename="package://amr_mtt/meshes/amr_mtt_model/F_Cam_Link.STL" scale="1 1 1"/>
                 </geometry>
                 <material name="red">

Commit message: update backup

File: urdf/amr_mtt.xacro (robot description, xacro)
@@ -47,4 +47,16 @@
     <xacro:arg name="odometry_source" default="world" />
     <xacro:property name="odometry_source" value="$(arg odometry_source)"/>
+    <!-- UR5 Robot -->
+    <xacro:include filename="$(find ur_description)/urdf/ur_macro.xacro"/>
+    <xacro:arg name="ur_type" default="ur5"/>
+    <xacro:arg name="joint_limit_params" default="$(find ur_description)/config/ur5/joint_limits.yaml"/>
+    <xacro:arg name="kinematics_params" default="$(find ur_description)/config/ur5/default_kinematics.yaml"/>
+    <xacro:arg name="physical_params" default="$(find ur_description)/config/ur5/physical_parameters.yaml"/>
+    <xacro:arg name="visual_params" default="$(find ur_description)/config/ur5/visual_parameters.yaml"/>
+    <!-- <xacro:arg name="initial_positions_file" default="$(find ur_description)/config/ur5/initial_positions.yaml"/> -->
+    <xacro:arg name="initial_positions_file" default="$(find amr_mtt)/config/initial_positions.yaml"/>
+    <xacro:property name="initial_positions_file" value="$(arg initial_positions_file)"/>
+    <!--Gripper-->
+    <!-- <xacro:include filename="$(find robotiq_description)/urdf/robotiq_2f_85_macro.urdf.xacro" /> -->
     <!-- ............................... LOAD MACROS ................................. -->
     <xacro:include filename="$(find amr_mtt)/urdf/materials.xacro"/>
@@ -95,4 +107,26 @@
         <origin xyz="0.0 0 0" rpy="0 0 0.0" />
     </joint>
+    <!-- ................................ UR5 ROBOT ARM .......................... -->
+    <xacro:ur_robot
+        name="ur5_arm"
+        tf_prefix="ur5_"
+        parent="base_link"
+        joint_limits_parameters_file="$(arg joint_limit_params)"
+        kinematics_parameters_file="$(arg kinematics_params)"
+        physical_parameters_file="$(arg physical_params)"
+        visual_parameters_file="$(arg visual_params)"
+        use_fake_hardware="false"
+        sim_ignition="true"
+        initial_positions="${xacro.load_yaml(initial_positions_file)}"
+    >
+        <origin xyz="0.2 0 0.8" rpy="0 0 0"/>
+    </xacro:ur_robot>
+    <!-- ................................ ROBOTIQ GRIPPER .......................... -->
+    <!-- <xacro:robotiq_gripper
+        name="robotiq_gripper"
+        prefix=""
+        parent="ur5_tool0"
+        include_ros2_control="false">  <origin xyz="0 0 0" rpy="0 0 0"/>
+    </xacro:robotiq_gripper> -->
     <!-- ................................ WHEELS ..................................... -->
     <xacro:trolley_wheel cardinality="front" dexterity="left" origin_x="${chassis_length/2-0.10}" origin_y="${trolley_track_width/2}" origin_z="-${trolley_wheel_radius+chassis_height/2}"/>

File: urdf/ign.xacro (robot description, xacro)
@@ -29,4 +29,12 @@
             <child_frame_id>base_footprint</child_frame_id>
         </plugin>
+    </gazebo>
+    <gazebo>
+        <plugin filename="ign_ros2_control-system" name="ign_ros2_control::IgnitionROS2ControlPlugin">
+            <parameters>$(find amr_mtt)/config/ur5_controllers.yaml</parameters>
+        </plugin>
+    </gazebo>
+    <gazebo reference="ur5_base_link">
+        <self_collide>true</self_collide>
     </gazebo>
     <!-- ............................. ground truth .................................... -->

Commit message: update battery node
update update battery but not test

File: urdf/amr_mtt.xacro (robot description, xacro)
@@ -12,5 +12,6 @@
     <xacro:property name="traction_max_wheel_torque" value="11.4"/>
     <xacro:property name="traction_wheel_friction" value="3.0"/>
-    <xacro:property name="trolley_wheel_mass" value="0.1"/>
+    <!-- trolley_wheel_mass (มวลของล้อเลื่อน) เพิ่มน้ำหนักล้อประคอง (Mass) unit Kg -->
+    <xacro:property name="trolley_wheel_mass" value="2.0"/>
     <xacro:property name="trolley_track_width" value="0.5"/>
     <xacro:property name="trolley_wheel_friction" value="0.0"/>
@@ -107,4 +108,33 @@
         <origin xyz="0.0 0 0" rpy="0 0 0.0" />
     </joint>
+    <!-- ========================================= battery_ =========================================== -->
+    <link name="battery_link">
+        <visual>
+            <origin xyz="0 0 0" rpy="0 0 0"/>
+            <geometry>
+                <box size="0.2 0.3 0.15"/> </geometry>
+            <material name="black"/>
+        </visual>
+        <collision>
+            <origin xyz="0 0 0" rpy="0 0 0"/>
+            <geometry>
+                <box size="0.2 0.3 0.15"/>
+            </geometry>
+        </collision>
+        <inertial>
+            <origin xyz="0 0 0" rpy="0 0 0"/>
+            <mass value="20.0"/>
+            <xacro:box_inertia m="20.0" x="0.2" y="0.3" z="0.15"/>
+        </inertial>
+    </link>
+    <joint name="battery_joint" type="fixed">
+        <parent link="base_link"/>
+        <child link="battery_link"/>
+        <origin xyz="-0.35 0 ${chassis_height/2 + 0.075}" rpy="0 0 0"/>
+    </joint>
+    <gazebo reference="battery_link">
+        <material>Gazebo/DarkGrey</material>
+    </gazebo>
+    <!-- ============================================================================= -->
     <!-- ................................ UR5 ROBOT ARM .......................... -->
     <xacro:ur_robot

File: urdf/ign.xacro (robot description, xacro)
@@ -10,32 +10,39 @@
         <plugin filename="ignition-gazebo-joint-state-publisher-system" name="ignition::gazebo::systems::JointStatePublisher">
         </plugin>
-        <!-- ........................... DIFFERENTIAL DRIVE PLUGIN ................................... -->
-        <plugin filename="ignition-gazebo-diff-drive-system" name="ignition::gazebo::systems::DiffDrive">
-            <left_joint>middle_left_wheel_joint</left_joint>
-            <right_joint>middle_right_wheel_joint</right_joint>
-            <wheel_separation>${traction_track_width}</wheel_separation>
-            <wheel_radius>${traction_wheel_radius}</wheel_radius>
-            <odom_publish_frequency>50</odom_publish_frequency>
-            <topic>/cmd_vel</topic>
-            <max_linear_acceleration>0.8</max_linear_acceleration>
-            <max_angular_acceleration>2.0</max_angular_acceleration>
-            <min_linear_acceleration>-0.8</min_linear_acceleration>
-            <min_angular_acceleration>-2.0</min_angular_acceleration>
-            <xacro:if value="${odometry_source == 'encoders'}">
-                <odom_topic>$(arg wheel_odom_topic)</odom_topic>
-                <tf_topic>/tf</tf_topic>
-            </xacro:if>
-            <frame_id>odom</frame_id>
-            <child_frame_id>base_footprint</child_frame_id>
-        </plugin>
-    </gazebo>
+    </gazebo>
+    <!-- ........................... ROS2 CONTROL PLUGIN ................................... -->
     <gazebo>
         <plugin filename="ign_ros2_control-system" name="ign_ros2_control::IgnitionROS2ControlPlugin">
-            <parameters>$(find amr_mtt)/config/ur5_controllers.yaml</parameters>
-        </plugin>
-    </gazebo>
-    <gazebo reference="ur5_base_link">
-        <self_collide>true</self_collide>
-    </gazebo>
+            <parameters>$(find amr_mtt)/config/controllers.yaml</parameters>
+        </plugin>
+    </gazebo>
+    <ros2_control name="MobileBase" type="system">
+        <hardware>
+            <plugin>ign_ros2_control/IgnitionSystem</plugin>
+        </hardware>
+        <joint name="middle_left_wheel_joint">
+            <command_interface name="velocity"/>
+            <state_interface name="position"/>
+            <state_interface name="velocity"/>
+        </joint>
+        <joint name="middle_right_wheel_joint">
+            <command_interface name="velocity"/>
+            <state_interface name="position"/>
+            <state_interface name="velocity"/>
+        </joint>
+    </ros2_control>
+    <!--======================================= linearbattery ================================================ -->
+    <plugin filename="ignition-gazebo-linearbattery-system" name="ignition::gazebo::systems::LinearBatteryPlugin">
+        <battery_name>linear_battery</battery_name>
+        <voltage>24.0</voltage>
+        <open_circuit_voltage_constant_coef>24.0</open_circuit_voltage_constant_coef>
+        <open_circuit_voltage_linear_coef>-3.0</open_circuit_voltage_linear_coef>
+        <initial_charge>100.0</initial_charge>
+        <capacity>100.0</capacity>
+        <resistance>0.072</resistance>
+        <smooth_current_tau>2.0</smooth_current_tau>
+        <power_load>100.0</power_load>
+        <soc_threshold>0.10</soc_threshold>
+    </plugin>
     <!-- ............................. ground truth .................................... -->
     <xacro:if value="${odometry_source == 'world'}">
@@ -52,4 +59,5 @@
     </xacro:if>
     <!-- ........................... 2D LIDAR config ................................... -->
+    <!-- ====================== Font LiDAR ======================== -->
     <xacro:if value="$(arg two_d_lidar_enabled)">
         <gazebo reference="L_F_Lidar_Link">
@@ -187,4 +195,10 @@
         </gazebo>
     </xacro:if>
+    <!-- ============================================= ur5 ===================================== -->
+    <gazebo reference="ur5_base_link">
+        <!-- คำสั่ง <self_collide>true</self_collide> เป็นการบอก Gazebo ว่า "ช่วยเช็คหน่อยนะ
+            ถ้าชิ้นส่วน ur5_base_link (ฐานแขน) ไปโดนชิ้นส่วนอื่นของหุ่นยนต์ตัวเดียวกัน ให้ถือว่า ชนกัน (ห้ามทะลุผ่าน) -->
+        <self_collide>true</self_collide>
+    </gazebo>
     <!-- ........................... MATERIALS ................................... -->
     <gazebo reference="base_link">

Commit message: Update amr_mtt.xacro

File: urdf/amr_mtt.xacro (robot description, xacro)
@@ -260,5 +260,5 @@
                     <mesh filename="package://amr_mtt/meshes/amr_mtt_model/F_Cam_Link.STL" scale="1 1 1"/>
                 </geometry>
-                <material name="blue">
+                <material name="black">
                     <color rgba="0 0 1 1" />
                 </material>
