Commit message: update
update

File: urdf/amr_mtt.xacro (robot description, xacro)
@@ -11,5 +11,5 @@
     <xacro:property name="traction_wheel_base" value="0.88"/>
     <xacro:property name="traction_max_wheel_torque" value="11.4"/>
-    <xacro:property name="traction_wheel_friction" value="3.0"/>
+    <xacro:property name="traction_wheel_friction" value="5.0"/>
     <!-- trolley_wheel_mass (มวลของล้อเลื่อน) เพิ่มน้ำหนักล้อประคอง (Mass) unit Kg -->
     <xacro:property name="trolley_wheel_mass" value="2.0"/>
@@ -78,5 +78,5 @@
         <parent link="base_footprint"/>
         <child link="base_link"/>
-        <origin xyz="0.0 0 ${chassis_height/2 + traction_wheel_radius}" rpy="0 0 0.0" />
+        <origin xyz="0.0 0 ${chassis_height/2 + 2*trolley_wheel_radius + eps}" rpy="0 0 0.0" />
     </joint>
     <link name="chassis_link">
@@ -164,6 +164,6 @@
     <xacro:trolley_wheel cardinality="back" dexterity="left" origin_x="-${chassis_length/2-0.10}" origin_y="${trolley_track_width/2}" origin_z="-${trolley_wheel_radius+chassis_height/2}"/>
     <xacro:trolley_wheel cardinality="back" dexterity="right" origin_x="-${chassis_length/2-0.10}" origin_y="-${trolley_track_width/2}" origin_z="-${trolley_wheel_radius+chassis_height/2}"/>
-    <xacro:traction_wheel cardinality="middle" dexterity="left" origin_x="0" origin_y="${traction_track_width/2}" origin_z="-${chassis_height/2+2*trolley_wheel_radius+eps-traction_wheel_radius}"/>
-    <xacro:traction_wheel cardinality="middle" dexterity="right" origin_x="0" origin_y="-${traction_track_width/2}" origin_z="-${chassis_height/2+2*trolley_wheel_radius+eps-traction_wheel_radius}"/>
+    <xacro:traction_wheel cardinality="middle" dexterity="left" origin_x="0" origin_y="${traction_track_width/2}" origin_z="-${chassis_height/2+2*trolley_wheel_radius+eps-traction_wheel_radius}" friction="${traction_wheel_friction}"/>
+    <xacro:traction_wheel cardinality="middle" dexterity="right" origin_x="0" origin_y="-${traction_track_width/2}" origin_z="-${chassis_height/2+2*trolley_wheel_radius+eps-traction_wheel_radius}" friction="${traction_wheel_friction}"/>
     <!-- ............................. 2D LIDAR ........................................ -->
     <!-- ========================================================= -->
@@ -281,4 +281,40 @@
         </joint>
     </xacro:if>
+    <!-- ............................. REAR CAMERA ........................................ -->
+    <xacro:if value="$(arg camera_enabled)">
+        <!-- REAR CAMERA -->
+        <link name="rear_camera">
+            <collision>
+                <origin xyz="0 0 0" rpy="0 0 0" />
+                <geometry>
+                    <mesh filename="package://amr_mtt/meshes/amr_mtt_model/F_Cam_Link.STL" scale="1 1 1"/>
+                </geometry>
+            </collision>
+            <visual>
+                <origin xyz="0 0 0" rpy="0 0 0" />
+                <geometry>
+                    <mesh filename="package://amr_mtt/meshes/amr_mtt_model/F_Cam_Link.STL" scale="1 1 1"/>
+                </geometry>
+                <material name="black">
+                    <color rgba="1 0 0 1" />
+                </material>
+            </visual>
+            <inertial>
+                <mass value="0.01"/>
+                <xacro:box_inertia m="0.01" x="0.07" y="0.3" z = "0.09"/>
+            </inertial>
+        </link>
+        <joint name="rear_camera_joint" type="fixed">
+            <origin rpy="0 0 ${pi}" xyz="${-chassis_length/2} 0 0.26"/>
+            <parent link="base_link"/>
+            <child link="rear_camera"/>
+        </joint>
+        <link name="rear_camera_optical"/>
+        <joint name="rear_camera_optical_joint" type="fixed">
+            <origin xyz="0 0 0" rpy="${-pi/2} 0 ${-pi/2}"/>
+            <parent link="rear_camera"/>
+            <child link="rear_camera_optical"/>
+        </joint>
+    </xacro:if>
     <!-- .............................STEREO CAMERA ........................................ -->
     <xacro:if value="$(arg stereo_camera_enabled)">

File: urdf/ign.xacro (robot description, xacro)
@@ -12,4 +12,6 @@
     </gazebo>
     <!-- ........................... ROS2 CONTROL PLUGIN ................................... -->
+    <!-- ........................... ROS2 CONTROL PLUGIN ................................... -->
+    <!-- Enable plugin loader to support UR5 Arm (even if MobileBase is disabled here) -->
     <gazebo>
         <plugin filename="ign_ros2_control-system" name="ign_ros2_control::IgnitionROS2ControlPlugin">
@@ -17,4 +19,5 @@
         </plugin>
     </gazebo>
+    <!-- Enable MobileBase Control (Use ros2_control) -->
     <ros2_control name="MobileBase" type="system">
         <hardware>
@@ -32,7 +35,24 @@
         </joint>
     </ros2_control>
+    <!-- Disable Native DiffDrive Plugin (Using ros2_control instead) -->
+    <!-- <gazebo>
+        <plugin
+            filename="ignition-gazebo-diff-drive-system"
+            name="ignition::gazebo::systems::DiffDrive">
+            <left_joint>middle_left_wheel_joint</left_joint>
+            <right_joint>middle_right_wheel_joint</right_joint>
+            <wheel_separation>0.436</wheel_separation>
+            <wheel_radius>0.08</wheel_radius>
+            <odom_publish_frequency>50</odom_publish_frequency>
+            <topic>/cmd_vel</topic>
+            <odom_topic>odom</odom_topic>
+            <tf_topic>tf</tf_topic>
+            <frame_id>odom</frame_id>
+            <child_frame_id>base_footprint</child_frame_id>
+        </plugin>
+    </gazebo> -->
     <!--======================================= linearbattery ================================================ -->
     <gazebo>
-        <plugin filename="libignition-gazebo-linearbattery-system.so" name="ignition::gazebo::systems::LinearBatteryPlugin">
+        <plugin filename="libignition-gazebo-linearbatteryplugin-system.so" name="ignition::gazebo::systems::LinearBatteryPlugin">
             <battery_name>linear_battery</battery_name>
             <voltage>24.0</voltage>
@@ -126,9 +146,32 @@
     <xacro:if value="$(arg camera_enabled)">
         <gazebo reference="kinect_camera">
-            <sensor type="depth_camera" name="kinect_camera">
+            <sensor type="camera" name="kinect_camera">
                 <update_rate>30.0</update_rate>
                 <topic>kinect_camera</topic>
                 <ignition_frame_id>kinect_camera</ignition_frame_id>
                 <camera_info_topic>kinect_camera/camera_info</camera_info_topic>
+                <camera>
+                    <horizontal_fov>${radians(camera_horizontal_fov)}</horizontal_fov>
+                    <image>
+                        <width>640</width>
+                        <height>480</height>
+                        <format>R8G8B8</format>
+                    </image>
+                    <clip>
+                        <near>0.05</near>
+                        <far>8.0</far>
+                    </clip>
+                </camera>
+            </sensor>
+        </gazebo>
+    </xacro:if>
+    <!-- ........................... REAR CAMERA config ................................... -->
+    <xacro:if value="$(arg camera_enabled)">
+        <gazebo reference="rear_camera">
+            <sensor type="camera" name="rear_camera">
+                <update_rate>30.0</update_rate>
+                <topic>rear_camera</topic>
+                <ignition_frame_id>rear_camera</ignition_frame_id>
+                <camera_info_topic>rear_camera/camera_info</camera_info_topic>
                 <camera>
                     <horizontal_fov>${radians(camera_horizontal_fov)}</horizontal_fov>

File: urdf/macros.xacro (robot description, xacro)
@@ -14,4 +14,48 @@
     <xacro:macro name="trolley_wheel" params="cardinality dexterity origin_x origin_y origin_z">
         <link name="${cardinality}_${dexterity}_wheel">
+            <visual name="${cardinality}_${dexterity}_bracket_visual">
+                <origin xyz="0 0 0" rpy="0 0 0" />
+                <geometry>
+                    <!-- Front Left -->
+                    <xacro:if value="${cardinality == 'front' and dexterity == 'left'}">
+                         <mesh filename="package://amr_mtt/meshes/amr_mtt_model/L_F_CasterBraket_Link.STL" scale="1 1 1"/>
+                    </xacro:if>
+                    <!-- Front Right -->
+                    <xacro:if value="${cardinality == 'front' and dexterity == 'right'}">
+                         <mesh filename="package://amr_mtt/meshes/amr_mtt_model/R_F_CasterBraket_Link.STL" scale="1 1 1"/>
+                    </xacro:if>
+                    <!-- Back Left -->
+                    <xacro:if value="${cardinality == 'back' and dexterity == 'left'}">
+                         <mesh filename="package://amr_mtt/meshes/amr_mtt_model/L_B_CasterBraket_Link.STL" scale="1 1 1"/>
+                    </xacro:if>
+                    <!-- Back Right -->
+                    <xacro:if value="${cardinality == 'back' and dexterity == 'right'}">
+                         <mesh filename="package://amr_mtt/meshes/amr_mtt_model/R_B_CasterBraket_Link.STL" scale="1 1 1"/>
+                    </xacro:if>
+                </geometry>
+                <material name="black"/>
+            </visual>
+            <visual name="${cardinality}_${dexterity}_wheel_visual">
+                <origin xyz="0 0 0" rpy="0 0 0" />
+                <geometry>
+                    <!-- Front Left -->
+                    <xacro:if value="${cardinality == 'front' and dexterity == 'left'}">
+                         <mesh filename="package://amr_mtt/meshes/amr_mtt_model/L_F_Caster_Wheel_Link.STL" scale="1 1 1"/>
+                    </xacro:if>
+                    <!-- Front Right -->
+                    <xacro:if value="${cardinality == 'front' and dexterity == 'right'}">
+                         <mesh filename="package://amr_mtt/meshes/amr_mtt_model/R_F_Caster_Wheel_Link.STL" scale="1 1 1"/>
+                    </xacro:if>
+                    <!-- Back Left -->
+                    <xacro:if value="${cardinality == 'back' and dexterity == 'left'}">
+                         <mesh filename="package://amr_mtt/meshes/amr_mtt_model/L_B_Caster_Wheel_Link.STL" scale="1 1 1"/>
+                    </xacro:if>
+                    <!-- Back Right -->
+                    <xacro:if value="${cardinality == 'back' and dexterity == 'right'}">
+                         <mesh filename="package://amr_mtt/meshes/amr_mtt_model/R_B_Caster_Wheel_Link.STL" scale="1 1 1"/>
+                    </xacro:if>
+                </geometry>
+                <material name="black"/>
+            </visual>
             <collision>
                 <origin xyz="0 0 0" rpy="0 ${pi/2} ${pi/2}" />
@@ -37,5 +81,5 @@
         </gazebo>
     </xacro:macro>
-    <xacro:macro name="traction_wheel" params="cardinality dexterity origin_x origin_y origin_z">
+    <xacro:macro name="traction_wheel" params="cardinality dexterity origin_x origin_y origin_z friction">
         <link name="${cardinality}_${dexterity}_wheel">
             <collision>
@@ -46,4 +90,16 @@
                 <self_collide>false</self_collide>
             </collision>
+            <visual>
+                <origin xyz="0 0 0" rpy="0 0 0" />
+                <geometry>
+                    <xacro:if value="${dexterity == 'left'}">
+                        <mesh filename="package://amr_mtt/meshes/amr_mtt_model/L_Wheel_Link.STL" scale="1 1 1"/>
+                    </xacro:if>
+                    <xacro:if value="${dexterity == 'right'}">
+                        <mesh filename="package://amr_mtt/meshes/amr_mtt_model/R_Wheel_Link.STL" scale="1 1 1"/>
+                    </xacro:if>
+                </geometry>
+                <material name="black"/>
+            </visual>
             <inertial>
                 <origin xyz="0 0 0" rpy="0 ${pi/2} ${pi/2}" />
@@ -51,5 +107,5 @@
                 <xacro:cylinder_inertia m="${traction_wheel_mass}" r="${traction_wheel_radius}" h="${traction_wheel_width}"/>
             </inertial>
-            <mu>5.0</mu>
+            <mu>${friction}</mu>
         </link>
         <joint name="${cardinality}_${dexterity}_wheel_joint" type="continuous">
