Commit message: update
update

File: amr_mtt_bot/robotiq_description/urdf/robotiq_2f_85_macro.urdf.xacro (robot description, xacro)
@@ -226,12 +226,9 @@
             <dynamics damping="0.1" friction="0.1"/>
         </joint>
-        <joint name="${prefix}robotiq_85_right_knuckle_joint" type="revolute">
+        <joint name="${prefix}robotiq_85_right_knuckle_joint" type="fixed">
             <parent link="${prefix}robotiq_85_base_link" />
             <child link="${prefix}robotiq_85_right_knuckle_link" />
-            <axis xyz="0 -1 0" />
             <origin xyz="-0.03060114 0.0 0.05490452" rpy="0 0 0" />
-            <limit lower="-0.8" upper="0.0" velocity="0.5" effort="50" />
-            <mimic joint="${prefix}robotiq_85_left_knuckle_joint" multiplier="-1" />
-            <dynamics damping="0.1" friction="0.1"/>
+            <!-- FIXED: mimic ไม่ทำงานใน Ignition Gazebo -->
         </joint>
         <joint name="${prefix}robotiq_85_left_finger_joint" type="fixed">
@@ -245,35 +242,27 @@
             <origin xyz="-0.03152616 0.0 -0.00376347" rpy="0 0 0" />
         </joint>
-        <joint name="${prefix}robotiq_85_left_inner_knuckle_joint" type="continuous">
+        <joint name="${prefix}robotiq_85_left_inner_knuckle_joint" type="fixed">
             <parent link="${prefix}robotiq_85_base_link" />
             <child link="${prefix}robotiq_85_left_inner_knuckle_link" />
-            <axis xyz="0 -1 0" />
             <origin xyz="0.0127 0.0 0.06142" rpy="0 0 0" />
-            <mimic joint="${prefix}robotiq_85_left_knuckle_joint" />
-            <dynamics damping="0.1" friction="0.1"/>
-        </joint>
-        <joint name="${prefix}robotiq_85_right_inner_knuckle_joint" type="continuous">
+            <!-- FIXED: mimic ไม่ทำงานใน Ignition Gazebo -->
+        </joint>
+        <joint name="${prefix}robotiq_85_right_inner_knuckle_joint" type="fixed">
             <parent link="${prefix}robotiq_85_base_link" />
             <child link="${prefix}robotiq_85_right_inner_knuckle_link" />
-            <axis xyz="0 -1 0" />
             <origin xyz="-0.0127 0.0 0.06142" rpy="0 0 0" />
-            <mimic joint="${prefix}robotiq_85_left_knuckle_joint" multiplier="-1" />
-            <dynamics damping="0.1" friction="0.1"/>
-        </joint>
-        <joint name="${prefix}robotiq_85_left_finger_tip_joint" type="continuous">
+            <!-- FIXED: mimic ไม่ทำงานใน Ignition Gazebo -->
+        </joint>
+        <joint name="${prefix}robotiq_85_left_finger_tip_joint" type="fixed">
             <parent link="${prefix}robotiq_85_left_finger_link" />
             <child link="${prefix}robotiq_85_left_finger_tip_link" />
-            <axis xyz="0 -1 0" />
             <origin xyz="0.00563134 0.0 0.04718515" rpy="0 0 0" />
-            <mimic joint="${prefix}robotiq_85_left_knuckle_joint" multiplier="-1" />
-            <dynamics damping="0.1" friction="0.1"/>
-        </joint>
-        <joint name="${prefix}robotiq_85_right_finger_tip_joint" type="continuous">
+            <!-- FIXED: mimic ไม่ทำงานใน Ignition Gazebo -->
+        </joint>
+        <joint name="${prefix}robotiq_85_right_finger_tip_joint" type="fixed">
             <parent link="${prefix}robotiq_85_right_finger_link" />
             <child link="${prefix}robotiq_85_right_finger_tip_link" />
-            <axis xyz="0 -1 0" />
             <origin xyz="-0.00563134 0.0 0.04718515" rpy="0 0 0" />
-            <mimic joint="${prefix}robotiq_85_left_knuckle_joint" />
-            <dynamics damping="0.1" friction="0.1"/>
+            <!-- FIXED: mimic ไม่ทำงานใน Ignition Gazebo -->
         </joint>
     </xacro:macro>

File: amr_mtt_bot/urdf/amr_mtt.xacro (robot description, xacro)
@@ -6,5 +6,5 @@
     <xacro:property name="chassis_length" value="0.9"/>
     <xacro:property name="chassis_width" value="0.64"/>
-    <xacro:property name="chassis_height" value="0.2"/>
+    <xacro:property name="chassis_height" value="0.45"/>
     <!-- traction_wheel_mass (มวลของล้อขับเคลื่อน) -->
     <xacro:property name="traction_wheel_mass" value="4.6"/>
@@ -83,5 +83,5 @@
     <link name="chassis_link">
         <collision>
-            <origin xyz="0 0 -0.05" rpy="0 0 0" />
+            <origin xyz="0 0 0.025" rpy="0 0 0" />
             <geometry>
                 <box size="${chassis_length} ${chassis_width} ${chassis_height}"/>

File: amr_mtt_bot/urdf/ign.xacro (robot description, xacro)
@@ -289,4 +289,25 @@
             <state_interface name="velocity"/>
         </joint>
+        <!-- Mimic joints state interfaces for RViz -->
+        <joint name="robotiq_85_right_knuckle_joint">
+            <state_interface name="position"/>
+            <state_interface name="velocity"/>
+        </joint>
+        <joint name="robotiq_85_left_inner_knuckle_joint">
+            <state_interface name="position"/>
+            <state_interface name="velocity"/>
+        </joint>
+        <joint name="robotiq_85_right_inner_knuckle_joint">
+            <state_interface name="position"/>
+            <state_interface name="velocity"/>
+        </joint>
+        <joint name="robotiq_85_left_finger_tip_joint">
+            <state_interface name="position"/>
+            <state_interface name="velocity"/>
+        </joint>
+        <joint name="robotiq_85_right_finger_tip_joint">
+            <state_interface name="position"/>
+            <state_interface name="velocity"/>
+        </joint>
     </ros2_control>
 </robot>
