Commit message: update

File: amr_mtt_bot/urdf/amr_mtt.xacro (robot description, xacro)
@@ -3,5 +3,5 @@
     <!--................................ XACRO CONSTANTS .............................. -->
     <!-- หุ่นยนต์หนัก 60 kg -->
-    <xacro:property name="chassis_mass" value="135"/>
+    <xacro:property name="chassis_mass" value="60"/>
     <xacro:property name="chassis_length" value="0.9"/>
     <xacro:property name="chassis_width" value="0.64"/>
@@ -16,5 +16,5 @@
     <xacro:property name="trolley_track_width" value="0.5"/>
     <xacro:property name="trolley_wheel_friction" value="0.0"/>
-    <xacro:property name="trolley_wheel_radius" value="0.06"/>
+    <xacro:property name="trolley_wheel_radius" value="0.04"/>
     <!-- a small constant -->
     <xacro:property name="eps" value="0.001"/>
@@ -78,5 +78,6 @@
         <parent link="base_footprint"/>
         <child link="base_link"/>
-        <origin xyz="0.0 0 ${chassis_height/2 + 2*trolley_wheel_radius + eps}" rpy="0 0 0.0" />
+        <!-- Lift base_link by exactly 0.177m so the wheels touch the ground without sinking -->
+        <origin xyz="0.0 0 0.177" rpy="0 0 0.0" />
     </joint>
     <link name="chassis_link">
@@ -106,5 +107,5 @@
         <parent link="base_link"/>
         <child link="chassis_link"/>
-        <origin xyz="0.0 0 0" rpy="0 0 0.0" />
+        <origin xyz="0 0 0" rpy="0 0 0" />
     </joint>
     <!-- ========================================= battery_ =========================================== -->
@@ -150,5 +151,5 @@
         initial_positions="${xacro.load_yaml(initial_positions_file)}"
     >
-        <origin xyz="0.2 0 0.8" rpy="0 0 0"/>
+        <origin xyz="0.2 0 0.8755" rpy="0 0 0"/>
     </xacro:ur_robot>
     <!-- ................................ ROBOTIQ GRIPPER .......................... -->
@@ -160,10 +161,10 @@
     </xacro:robotiq_gripper>
     <!-- ................................ WHEELS ..................................... -->
-    <xacro:trolley_wheel cardinality="front" dexterity="left" origin_x="${chassis_length/2-0.10}" origin_y="${trolley_track_width/2}" origin_z="-${trolley_wheel_radius+chassis_height/2}"/>
-    <xacro:trolley_wheel cardinality="front" dexterity="right" origin_x="${chassis_length/2-0.10}" origin_y="-${trolley_track_width/2}" origin_z="-${trolley_wheel_radius+chassis_height/2}"/>
-    <xacro:trolley_wheel cardinality="back" dexterity="left" origin_x="-${chassis_length/2-0.10}" origin_y="${trolley_track_width/2}" origin_z="-${trolley_wheel_radius+chassis_height/2}"/>
-    <xacro:trolley_wheel cardinality="back" dexterity="right" origin_x="-${chassis_length/2-0.10}" origin_y="-${trolley_track_width/2}" origin_z="-${trolley_wheel_radius+chassis_height/2}"/>
-    <xacro:traction_wheel cardinality="middle" dexterity="left" origin_x="0" origin_y="${traction_track_width/2}" origin_z="-${chassis_height/2+2*trolley_wheel_radius+eps-traction_wheel_radius}" friction="${traction_wheel_friction}"/>
-    <xacro:traction_wheel cardinality="middle" dexterity="right" origin_x="0" origin_y="-${traction_track_width/2}" origin_z="-${chassis_height/2+2*trolley_wheel_radius+eps-traction_wheel_radius}" friction="${traction_wheel_friction}"/>
+    <xacro:trolley_wheel cardinality="front" dexterity="left" origin_x="0.31" origin_y="0.156" origin_z="-0.137"/>
+    <xacro:trolley_wheel cardinality="front" dexterity="right" origin_x="0.31" origin_y="-0.156" origin_z="-0.137"/>
+    <xacro:trolley_wheel cardinality="back" dexterity="left" origin_x="-0.31" origin_y="0.156" origin_z="-0.137"/>
+    <xacro:trolley_wheel cardinality="back" dexterity="right" origin_x="-0.31" origin_y="-0.156" origin_z="-0.137"/>
+    <xacro:traction_wheel cardinality="middle" dexterity="left" origin_x="0" origin_y="0.218" origin_z="-0.097" friction="${traction_wheel_friction}"/>
+    <xacro:traction_wheel cardinality="middle" dexterity="right" origin_x="0" origin_y="-0.218" origin_z="-0.097" friction="${traction_wheel_friction}"/>
     <!-- ............................. 2D LIDAR ........................................ -->
     <!-- ========================================================= -->

Commit message: update

File: amr_mtt_bot/urdf/amr_mtt.xacro (robot description, xacro)
@@ -25,5 +25,5 @@
     <xacro:property name="traction_wheel_width" value="0.06"/>
     <!-- พารามิเตอร์นี้คือระยะห่างระหว่าง "กึ่งกลางล้อซ้าย" ถึง "กึ่งกลางล้อขวา" -->
-    <xacro:property name="traction_track_width" value="0.436"/>
+    <xacro:property name="traction_track_width" value="0.5"/>
     <xacro:property name="two_d_lidar_update_rate" value="30"/>
     <xacro:property name="two_d_lidar_sample_size" value="361"/>
@@ -79,5 +79,5 @@
         <child link="base_link"/>
         <!-- Lift base_link by exactly 0.177m so the wheels touch the ground without sinking -->
-        <origin xyz="0.0 0 0.177" rpy="0 0 0.0" />
+        <origin xyz="0.0 0 0.25" rpy="0 0 0.0" />
     </joint>
     <link name="chassis_link">
@@ -89,10 +89,11 @@
         </collision>
         <visual>
-            <origin xyz="0 0 0" rpy="0 0 0" />
+            <!-- แก้ไขแกนกลับมาแนวนอน (Roll=0, Pitch=0), หมุนแกน Z (Yaw=90 องศา หรือ 1.5708) -->
+            <origin xyz="0 0 0.2" rpy="0 0 -1.5708" />
             <geometry>
                 <!-- <mesh filename="file://$(find amr_mtt_bot)/meshes/amr_mtt_model/base_link.STL" scale="1 1 1"/> -->
                 <mesh filename="package://amr_mtt_bot/meshes/amr_mtt_model/base_link.STL" scale="1 1 1"/>
             </geometry>
-            <material name="orange"/>
+            <material name="dark_grey"/>
         </visual>
        <inertial>
@@ -115,5 +116,7 @@
             <geometry>
                 <box size="0.2 0.3 0.15"/> </geometry>
-            <material name="black"/>
+            <material name="red">
+                <color rgba="1 0 0 1"/>
+            </material>
         </visual>
         <collision>
@@ -126,5 +129,5 @@
             <origin xyz="0 0 0" rpy="0 0 0"/>
             <mass value="20.0"/>
-            <xacro:box_inertia m="20.0" x="0.2" y="0.3" z="0.15"/>
+            <xacro:box_inertia m="20.0" x="0.15" y="0.25" z="0.10"/>
         </inertial>
     </link>
@@ -132,5 +135,5 @@
         <parent link="base_link"/>
         <child link="battery_link"/>
-        <origin xyz="-0.35 0 ${chassis_height/2 + 0.075}" rpy="0 0 0"/>
+        <origin xyz="-0.2 0 0.02" rpy="0 0 0"/>
     </joint>
     <gazebo reference="battery_link">
@@ -151,5 +154,5 @@
         initial_positions="${xacro.load_yaml(initial_positions_file)}"
     >
-        <origin xyz="0.2 0 0.8755" rpy="0 0 0"/>
+        <origin xyz="0.2 0 0.72" rpy="0 0 0"/>
     </xacro:ur_robot>
     <!-- ................................ ROBOTIQ GRIPPER .......................... -->
@@ -161,10 +164,10 @@
     </xacro:robotiq_gripper>
     <!-- ................................ WHEELS ..................................... -->
-    <xacro:trolley_wheel cardinality="front" dexterity="left" origin_x="0.31" origin_y="0.156" origin_z="-0.137"/>
-    <xacro:trolley_wheel cardinality="front" dexterity="right" origin_x="0.31" origin_y="-0.156" origin_z="-0.137"/>
-    <xacro:trolley_wheel cardinality="back" dexterity="left" origin_x="-0.31" origin_y="0.156" origin_z="-0.137"/>
-    <xacro:trolley_wheel cardinality="back" dexterity="right" origin_x="-0.31" origin_y="-0.156" origin_z="-0.137"/>
-    <xacro:traction_wheel cardinality="middle" dexterity="left" origin_x="0" origin_y="0.218" origin_z="-0.097" friction="${traction_wheel_friction}"/>
-    <xacro:traction_wheel cardinality="middle" dexterity="right" origin_x="0" origin_y="-0.218" origin_z="-0.097" friction="${traction_wheel_friction}"/>
+    <xacro:trolley_wheel cardinality="front" dexterity="left" origin_x="0.35" origin_y="0.25" origin_z="-0.21"/>
+    <xacro:trolley_wheel cardinality="front" dexterity="right" origin_x="0.35" origin_y="-0.25" origin_z="-0.21"/>
+    <xacro:trolley_wheel cardinality="back" dexterity="left" origin_x="-0.35" origin_y="0.25" origin_z="-0.21"/>
+    <xacro:trolley_wheel cardinality="back" dexterity="right" origin_x="-0.35" origin_y="-0.25" origin_z="-0.21"/>
+    <xacro:traction_wheel cardinality="middle" dexterity="left" origin_x="0" origin_y="0.28" origin_z="-0.17" friction="${traction_wheel_friction}"/>
+    <xacro:traction_wheel cardinality="middle" dexterity="right" origin_x="0" origin_y="-0.28" origin_z="-0.17" friction="${traction_wheel_friction}"/>
     <!-- ............................. 2D LIDAR ........................................ -->
     <!-- ========================================================= -->
@@ -184,6 +187,6 @@
                     <mesh filename="package://amr_mtt_bot/meshes/amr_mtt_model/L_F_Lidar_Link.STL" scale="1 1 1"/>
                 </geometry>
-                <material name="black">
-                    <color rgba="0 0 0 1" />
+                <material name="lidar_grey">
+                    <color rgba="0.706 0.706 0.706 1" />
                 </material>
             </visual>
@@ -197,8 +200,17 @@
             <parent link="base_link"/>
             <child link="L_F_Lidar_Link"/>
-            <origin xyz="0.33905 0.18905 0.18259" rpy="3.1416 0 0.7854"/>
-        </joint>
+            <origin xyz="0.4 0.25 0.07" rpy="3.1416 0 0.7854"/>
+        </joint>
+        <gazebo reference="L_F_Lidar_joint">
+            <preserveFixedJoint>true</preserveFixedJoint>
+        </gazebo>
         <gazebo reference="L_F_Lidar_Link">
-            <material>Gazebo/White</material>
+            <visual>
+                <material>
+                    <ambient>0.706 0.706 0.706 1.0</ambient>
+                    <diffuse>0.706 0.706 0.706 1.0</diffuse>
+                    <specular>0.706 0.706 0.706 1.0</specular>
+                </material>
+            </visual>
         </gazebo>
     </xacro:if>
@@ -219,6 +231,6 @@
                     <mesh filename="package://amr_mtt_bot/meshes/amr_mtt_model/R_B_Lidar_Link.STL" scale="1 1 1"/>
                 </geometry>
-                <material name="black">
-                    <color rgba="0 0 0 1" />
+                <material name="lidar_grey">
+                    <color rgba="0.706 0.706 0.706 1" />
                 </material>
             </visual>
@@ -233,12 +245,37 @@
             <child link="R_B_Lidar_Link"/>
             <!-- จุดติดตั้งด้านหลัง -->
-            <origin xyz="-0.33905 -0.18905 0.18259" rpy="-3.1416 0 -0.7854"/>
-        </joint>
+            <origin xyz="-0.4 -0.25 0.07" rpy="-3.1416 0 -0.7854"/>
+        </joint>
+        <gazebo reference="R_B_Lidar_joint">
+            <preserveFixedJoint>true</preserveFixedJoint>
+        </gazebo>
         <gazebo reference="R_B_Lidar_Link">
-            <material>Gazebo/White</material>
+            <visual>
+                <material>
+                    <ambient>0.706 0.706 0.706 1.0</ambient>
+                    <diffuse>0.706 0.706 0.706 1.0</diffuse>
+                    <specular>0.706 0.706 0.706 1.0</specular>
+                </material>
+            </visual>
         </gazebo>
     </xacro:if>
     <!-- ............................. IMU ........................................ -->
-    <link name="imu_frame"/>
+    <link name="imu_frame">
+        <collision>
+            <origin xyz="0 0 0.08" rpy="0 0 0" />
+            <geometry>
+                <mesh filename="package://amr_mtt_bot/meshes/amr_mtt_model/IMU_Link.STL" scale="1 1 1"/>
+            </geometry>
+         </collision>
+         <visual>
+            <origin xyz="0 0 0.08" rpy="0 0 0" />
+            <geometry>
+                <mesh filename="package://amr_mtt_bot/meshes/amr_mtt_model/IMU_Link.STL" scale="1 1 1"/>
+            </geometry>
+            <material name="blue">
+                <color rgba="0 0 0 1" />
+            </material>
+         </visual>
+    </link>
     <joint name="imu_joint" type="fixed">
         <parent link="base_link"/>
@@ -271,5 +308,5 @@
         </link>
         <joint name="kinect_camera_joint" type="fixed">
-            <origin rpy="0 0 0" xyz="${chassis_length/2} 0 0.26"/>
+            <origin rpy="0 0 0" xyz="${(chassis_length/2) + 0.03} 0 0.14"/>
             <parent link="base_link"/>
             <child link="kinect_camera"/>
@@ -307,5 +344,5 @@
         </link>
         <joint name="rear_camera_joint" type="fixed">
-            <origin rpy="0 0 ${pi}" xyz="${-chassis_length/2} 0 0.26"/>
+            <origin rpy="0 0 ${pi}" xyz="${-(chassis_length/2) - 0.03} 0 0.14"/>
             <parent link="base_link"/>
             <child link="rear_camera"/>
@@ -343,5 +380,5 @@
         </link>
         <joint name="stereo_camera_joint" type="fixed">
-            <origin rpy="0 0 0" xyz="${chassis_length/2} 0 0.26"/>
+            <origin rpy="0 0 0" xyz="${(chassis_length/2) + 0.03} 0 0.14"/>
             <parent link="base_link"/>
             <child link="stereo_camera"/>

File: amr_mtt_bot/urdf/ign.xacro (robot description, xacro)
@@ -76,5 +76,5 @@
                 <tf_topic>/tf</tf_topic>
                 <dimensions>2</dimensions>
-                <odom_publish_frequency>10</odom_publish_frequency>
+                <odom_publish_frequency>50</odom_publish_frequency>
             </plugin>
         </gazebo>

File: amr_mtt_bot/urdf/macros.xacro (robot description, xacro)
@@ -15,5 +15,5 @@
         <link name="${cardinality}_${dexterity}_wheel">
             <visual name="${cardinality}_${dexterity}_bracket_visual">
-                <origin xyz="0 0 0" rpy="0 0 0" />
+                <origin xyz="0 0 0.05" rpy="0 0 0" />
                 <geometry>
                     <!-- Front Left -->
@@ -34,5 +34,5 @@
                     </xacro:if>
                 </geometry>
-                <material name="black"/>
+                <material name="orange"/>
             </visual>
             <visual name="${cardinality}_${dexterity}_wheel_visual">
@@ -56,5 +56,5 @@
                     </xacro:if>
                 </geometry>
-                <material name="black"/>
+                <material name="orange"/>
             </visual>
             <collision>
@@ -78,5 +78,17 @@
         </joint>
         <gazebo reference="${cardinality}_${dexterity}_wheel">
-            <material>Gazebo/Black</material>
+            <visual>
+                <material>
+                    <ambient>0.8 0.4 0.0 1.0</ambient>
+                    <diffuse>0.8 0.4 0.0 1.0</diffuse>
+                    <specular>0.8 0.4 0.0 1.0</specular>
+                </material>
+            </visual>
+            <mu1>0.0</mu1>
+            <mu2>0.0</mu2>
+            <kp>10000000.0</kp>
+            <kd>1.0</kd>
+            <minDepth>0.001</minDepth>
+            <fdir1>1 0 0</fdir1>
         </gazebo>
     </xacro:macro>
@@ -100,5 +112,5 @@
                     </xacro:if>
                 </geometry>
-                <material name="black"/>
+                <material name="orange"/>
             </visual>
             <inertial>
@@ -116,5 +128,17 @@
         </joint>
         <gazebo reference="${cardinality}_${dexterity}_wheel">
-            <material>Gazebo/Black</material>
+            <visual>
+                <material>
+                    <ambient>0.3 0.3 0.3 1.0</ambient>
+                    <diffuse>0.3 0.3 0.3 1.0</diffuse>
+                    <specular>0.3 0.3 0.3 1.0</specular>
+                </material>
+            </visual>
+            <mu1>${friction}</mu1>
+            <mu2>${friction}</mu2>
+            <kp>10000000.0</kp>
+            <kd>1.0</kd>
+            <minDepth>0.001</minDepth>
+            <fdir1>1 0 0</fdir1>
         </gazebo>
     </xacro:macro>

Commit message: update

File: amr_mtt_bot/urdf/amr_mtt.xacro (robot description, xacro)
@@ -187,6 +187,6 @@
                     <mesh filename="package://amr_mtt_bot/meshes/amr_mtt_model/L_F_Lidar_Link.STL" scale="1 1 1"/>
                 </geometry>
-                <material name="lidar_grey">
-                    <color rgba="0.706 0.706 0.706 1" />
+                <material name="lidar_black">
+                    <color rgba="0.1 0.1 0.1 1" />
                 </material>
             </visual>
@@ -206,11 +206,5 @@
         </gazebo>
         <gazebo reference="L_F_Lidar_Link">
-            <visual>
-                <material>
-                    <ambient>0.706 0.706 0.706 1.0</ambient>
-                    <diffuse>0.706 0.706 0.706 1.0</diffuse>
-                    <specular>0.706 0.706 0.706 1.0</specular>
-                </material>
-            </visual>
+            <material>Gazebo/Black</material>
         </gazebo>
     </xacro:if>
@@ -231,6 +225,6 @@
                     <mesh filename="package://amr_mtt_bot/meshes/amr_mtt_model/R_B_Lidar_Link.STL" scale="1 1 1"/>
                 </geometry>
-                <material name="lidar_grey">
-                    <color rgba="0.706 0.706 0.706 1" />
+                <material name="lidar_black">
+                    <color rgba="0.1 0.1 0.1 1" />
                 </material>
             </visual>
@@ -251,11 +245,5 @@
         </gazebo>
         <gazebo reference="R_B_Lidar_Link">
-            <visual>
-                <material>
-                    <ambient>0.706 0.706 0.706 1.0</ambient>
-                    <diffuse>0.706 0.706 0.706 1.0</diffuse>
-                    <specular>0.706 0.706 0.706 1.0</specular>
-                </material>
-            </visual>
+            <material>Gazebo/Black</material>
         </gazebo>
     </xacro:if>

Commit message: Update amr_mtt.xacro

File: amr_mtt_bot/urdf/amr_mtt.xacro (robot description, xacro)
@@ -6,5 +6,5 @@
     <xacro:property name="chassis_length" value="0.9"/>
     <xacro:property name="chassis_width" value="0.64"/>
-    <xacro:property name="chassis_height" value="0.45"/>
+    <xacro:property name="chassis_height" value="0.40"/>
     <!-- traction_wheel_mass (มวลของล้อขับเคลื่อน) -->
     <xacro:property name="traction_wheel_mass" value="4.6"/>
@@ -83,5 +83,5 @@
     <link name="chassis_link">
         <collision>
-            <origin xyz="0 0 0.025" rpy="0 0 0" />
+            <origin xyz="0 0 0.0" rpy="0 0 0" />
             <geometry>
                 <box size="${chassis_length} ${chassis_width} ${chassis_height}"/>
