Commit message: update

File: amr_mtt_bot/urdf/amr_mtt.xacro (robot description, xacro)
@@ -2,6 +2,6 @@
 <robot xmlns:xacro="http://www.ros.org/wiki/xacro" name="amr_mtt">
     <!--................................ XACRO CONSTANTS .............................. -->
-    <!-- หุ่นยนต์หนัก 60 kg -->
-    <xacro:property name="chassis_mass" value="60"/>
+    <!-- หุ่นยนต์หนัก 200 kg รวมทุกชิ้นส่วน (chassis 162.8 + battery 20 + trolley wheels 8 + traction wheels 9.2) -->
+    <xacro:property name="chassis_mass" value="162.8"/>
     <xacro:property name="chassis_length" value="0.9"/>
     <xacro:property name="chassis_width" value="0.64"/>
@@ -26,13 +26,14 @@
     <!-- พารามิเตอร์นี้คือระยะห่างระหว่าง "กึ่งกลางล้อซ้าย" ถึง "กึ่งกลางล้อขวา" -->
     <xacro:property name="traction_track_width" value="0.5"/>
-    <xacro:property name="two_d_lidar_update_rate" value="30"/>
-    <xacro:property name="two_d_lidar_sample_size" value="361"/>
-    <xacro:property name="two_d_lidar_min_angle" value="0"/>
-    <xacro:property name="two_d_lidar_max_angle" value="360"/>
-    <xacro:property name="two_d_lidar_min_range" value="0.55"/>
-    <xacro:property name="two_d_lidar_max_range" value="16"/>
+    <!-- SICK picoScan100 : scanning angle 275° · resolution 0.1° · 50Hz · range 40m -->
+    <xacro:property name="two_d_lidar_update_rate" value="50"/>
+    <xacro:property name="two_d_lidar_sample_size" value="2750"/>
+    <xacro:property name="two_d_lidar_min_angle" value="-137.5"/>
+    <xacro:property name="two_d_lidar_max_angle" value="137.5"/>
+    <xacro:property name="two_d_lidar_min_range" value="0.35"/>
+    <xacro:property name="two_d_lidar_max_range" value="40"/>
     <xacro:property name="camera_baseline" value="0.06"/>
     <xacro:property name="camera_height" value="0.10"/>
-    <xacro:property name="camera_horizontal_fov" value="60"/>
+    <xacro:property name="camera_horizontal_fov" value="87"/>
     <xacro:arg name="robot_namespace" default=""/>
     <xacro:arg name="wheel_odom_topic" default="odom" />
@@ -239,5 +240,5 @@
             <child link="R_B_Lidar_Link"/>
             <!-- จุดติดตั้งด้านหลัง -->
-            <origin xyz="-0.4 -0.25 0.07" rpy="-3.1416 0 -0.7854"/>
+            <origin xyz="-0.4 -0.25 0.07" rpy="-3.1416 0 -2.3562"/>
         </joint>
         <gazebo reference="R_B_Lidar_joint">

File: amr_mtt_bot/urdf/ign.xacro (robot description, xacro)
@@ -11,5 +11,4 @@
         </plugin>
     </gazebo>
-    <!-- ........................... ROS2 CONTROL PLUGIN ................................... -->
     <!-- ........................... ROS2 CONTROL PLUGIN ................................... -->
     <!-- Enable plugin loader to support UR5 Arm (even if MobileBase is disabled here) -->
@@ -105,5 +104,5 @@
                         <type>gaussian</type>
                         <mean>0.0</mean>
-                        <stddev>0.001</stddev>
+                        <stddev>0.015</stddev>
                     </noise>
                 </lidar>
@@ -135,5 +134,5 @@
                         <type>gaussian</type>
                         <mean>0.0</mean>
-                        <stddev>0.001</stddev>
+                        <stddev>0.015</stddev>
                     </noise>
                 </lidar>
@@ -146,9 +145,8 @@
     <xacro:if value="$(arg camera_enabled)">
         <gazebo reference="kinect_camera">
-            <sensor type="camera" name="kinect_camera">
+            <sensor type="rgbd_camera" name="kinect_camera">
                 <update_rate>30.0</update_rate>
                 <topic>kinect_camera</topic>
                 <ignition_frame_id>kinect_camera</ignition_frame_id>
-                <camera_info_topic>kinect_camera/camera_info</camera_info_topic>
                 <camera>
                     <horizontal_fov>${radians(camera_horizontal_fov)}</horizontal_fov>
@@ -159,6 +157,6 @@
                     </image>
                     <clip>
-                        <near>0.05</near>
-                        <far>8.0</far>
+                        <near>0.1</near>
+                        <far>10.0</far>
                     </clip>
                 </camera>
@@ -169,9 +167,8 @@
     <xacro:if value="$(arg camera_enabled)">
         <gazebo reference="rear_camera">
-            <sensor type="camera" name="rear_camera">
+            <sensor type="rgbd_camera" name="rear_camera">
                 <update_rate>30.0</update_rate>
                 <topic>rear_camera</topic>
                 <ignition_frame_id>rear_camera</ignition_frame_id>
-                <camera_info_topic>rear_camera/camera_info</camera_info_topic>
                 <camera>
                     <horizontal_fov>${radians(camera_horizontal_fov)}</horizontal_fov>
@@ -182,6 +179,6 @@
                     </image>
                     <clip>
-                        <near>0.05</near>
-                        <far>8.0</far>
+                        <near>0.1</near>
+                        <far>10.0</far>
                     </clip>
                 </camera>
@@ -190,11 +187,58 @@
     </xacro:if>
     <!-- ........................... IMU config ................................... -->
+    <!-- Simulated as MicroStrain 3DM-GX5-10                                      -->
+    <!-- Gyro  ARW : 0.07 °/√hr  → σ = 0.0003 rad/s @ 200 Hz                    -->
+    <!-- Gyro  bias: 1 °/hr      → 4.85e-6 rad/s                                 -->
+    <!-- Accel VRW : 0.005 m/s/√hr → σ = 0.0012 m/s² @ 200 Hz                  -->
+    <!-- Accel bias: 0.025 mg    → 2.45e-4 m/s²                                  -->
     <gazebo reference="imu_frame">
         <sensor name="imu_sensor" type="imu">
             <always_on>1</always_on>
-            <update_rate>50</update_rate>
+            <update_rate>200</update_rate>
             <ignition_frame_id>imu_frame</ignition_frame_id>
             <visualize>true</visualize>
             <topic>imu</topic>
+            <imu>
+                <angular_velocity>
+                    <x><noise type="gaussian">
+                        <mean>0.0</mean>
+                        <stddev>0.0003</stddev>
+                        <bias_mean>0.0000049</bias_mean>
+                        <bias_stddev>0.0000025</bias_stddev>
+                    </noise></x>
+                    <y><noise type="gaussian">
+                        <mean>0.0</mean>
+                        <stddev>0.0003</stddev>
+                        <bias_mean>0.0000049</bias_mean>
+                        <bias_stddev>0.0000025</bias_stddev>
+                    </noise></y>
+                    <z><noise type="gaussian">
+                        <mean>0.0</mean>
+                        <stddev>0.0003</stddev>
+                        <bias_mean>0.0000049</bias_mean>
+                        <bias_stddev>0.0000025</bias_stddev>
+                    </noise></z>
+                </angular_velocity>
+                <linear_acceleration>
+                    <x><noise type="gaussian">
+                        <mean>0.0</mean>
+                        <stddev>0.0012</stddev>
+                        <bias_mean>0.000245</bias_mean>
+                        <bias_stddev>0.000125</bias_stddev>
+                    </noise></x>
+                    <y><noise type="gaussian">
+                        <mean>0.0</mean>
+                        <stddev>0.0012</stddev>
+                        <bias_mean>0.000245</bias_mean>
+                        <bias_stddev>0.000125</bias_stddev>
+                    </noise></y>
+                    <z><noise type="gaussian">
+                        <mean>0.0</mean>
+                        <stddev>0.0012</stddev>
+                        <bias_mean>0.000245</bias_mean>
+                        <bias_stddev>0.000125</bias_stddev>
+                    </noise></z>
+                </linear_acceleration>
+            </imu>
         </sensor>
     </gazebo>

Commit message: update

File: amr_mtt_bot/urdf/amr_mtt.xacro (robot description, xacro)
@@ -2,5 +2,5 @@
 <robot xmlns:xacro="http://www.ros.org/wiki/xacro" name="amr_mtt">
     <!--................................ XACRO CONSTANTS .............................. -->
-    <!-- หุ่นยนต์หนัก 200 kg รวมทุกชิ้นส่วน (chassis 162.8 + battery 20 + trolley wheels 8 + traction wheels 9.2) -->
+    <!-- หุ่นยนต์หนัก 200 kg -->
     <xacro:property name="chassis_mass" value="162.8"/>
     <xacro:property name="chassis_length" value="0.9"/>
@@ -287,6 +287,6 @@
                     <mesh filename="package://amr_mtt_bot/meshes/amr_mtt_model/F_Cam_Link.STL" scale="1 1 1"/>
                 </geometry>
-                <material name="black">
-                    <color rgba="0 0 1 1" />
+                <material name="white">
+                    <color rgba="1 1 1 1" />
                 </material>
             </visual>
@@ -323,6 +323,6 @@
                     <mesh filename="package://amr_mtt_bot/meshes/amr_mtt_model/F_Cam_Link.STL" scale="1 1 1"/>
                 </geometry>
-                <material name="black">
-                    <color rgba="1 0 0 1" />
+                <material name="white">
+                    <color rgba="1 1 1 1" />
                 </material>
             </visual>

File: amr_mtt_bot/urdf/ign.xacro (robot description, xacro)
@@ -143,4 +143,9 @@
     </xacro:if>
     <!-- ........................... CAMERA config ................................... -->
+    <!-- Simulated as Intel RealSense D435                                           -->
+    <!-- Depth H-FOV : 87°  V-FOV : 58°  (640×360 gives ~56° ≈ 58°)               -->
+    <!-- Depth Range : 0.1 m – 10.0 m                                               -->
+    <!-- Depth Noise : <2% at 2m  → stddev ≈ 0.007 m at 1m (Gaussian)             -->
+    <!-- RGB Update  : 30 Hz  (adequate for AMR navigation/mapping)                 -->
     <xacro:if value="$(arg camera_enabled)">
         <gazebo reference="kinect_camera">
@@ -150,8 +155,10 @@
                 <ignition_frame_id>kinect_camera</ignition_frame_id>
                 <camera>
+                    <!-- H-FOV 87° matches D435 depth module -->
                     <horizontal_fov>${radians(camera_horizontal_fov)}</horizontal_fov>
                     <image>
+                        <!-- 640×360 → V-FOV ≈ 56° (close to D435 58°) -->
                         <width>640</width>
-                        <height>480</height>
+                        <height>360</height>
                         <format>R8G8B8</format>
                     </image>
@@ -160,4 +167,10 @@
                         <far>10.0</far>
                     </clip>
+                    <!-- D435 depth noise: <2% at 2m → ~0.007 m stddev at 1m -->
+                    <noise>
+                        <type>gaussian</type>
+                        <mean>0.0</mean>
+                        <stddev>0.007</stddev>
+                    </noise>
                 </camera>
             </sensor>
@@ -175,5 +188,5 @@
                     <image>
                         <width>640</width>
-                        <height>480</height>
+                        <height>360</height>
                         <format>R8G8B8</format>
                     </image>
@@ -182,4 +195,9 @@
                         <far>10.0</far>
                     </clip>
+                    <noise>
+                        <type>gaussian</type>
+                        <mean>0.0</mean>
+                        <stddev>0.007</stddev>
+                    </noise>
                 </camera>
             </sensor>

Commit message: update Mar30 for last_version

File: amr_mtt_bot/urdf/amr_mtt.xacro (robot description, xacro)
@@ -33,5 +33,5 @@
     <xacro:property name="two_d_lidar_min_range" value="0.35"/>
     <xacro:property name="two_d_lidar_max_range" value="40"/>
-    <xacro:property name="camera_baseline" value="0.06"/>
+    <xacro:property name="camera_baseline" value="0.05"/>  <!-- D435 baseline = 50 mm -->
     <xacro:property name="camera_height" value="0.10"/>
     <xacro:property name="camera_horizontal_fov" value="87"/>

File: amr_mtt_bot/urdf/ign.xacro (robot description, xacro)
@@ -144,5 +144,5 @@
     <!-- ........................... CAMERA config ................................... -->
     <!-- Simulated as Intel RealSense D435                                           -->
-    <!-- Depth H-FOV : 87°  V-FOV : 58°  (640×360 gives ~56° ≈ 58°)               -->
+    <!-- Depth H-FOV : 87°  V-FOV : 58°  (640×480 gives ~58°)                     -->
     <!-- Depth Range : 0.1 m – 10.0 m                                               -->
     <!-- Depth Noise : <2% at 2m  → stddev ≈ 0.007 m at 1m (Gaussian)             -->
@@ -158,7 +158,7 @@
                     <horizontal_fov>${radians(camera_horizontal_fov)}</horizontal_fov>
                     <image>
-                        <!-- 640×360 → V-FOV ≈ 56° (close to D435 58°) -->
+                        <!-- 640×480 → V-FOV ≈ 58° matches D435 depth V-FOV -->
                         <width>640</width>
-                        <height>360</height>
+                        <height>480</height>
                         <format>R8G8B8</format>
                     </image>
@@ -187,6 +187,7 @@
                     <horizontal_fov>${radians(camera_horizontal_fov)}</horizontal_fov>
                     <image>
+                        <!-- 640×480 → V-FOV ≈ 58° matches D435 depth V-FOV -->
                         <width>640</width>
-                        <height>360</height>
+                        <height>480</height>
                         <format>R8G8B8</format>
                     </image>
@@ -262,40 +263,49 @@
     </gazebo>
     <!-- ........................... Stereo camera ................................... -->
+    <!-- Simulated as Intel RealSense D435 stereo IR pair                           -->
+    <!-- H-FOV : 87°  (1.5184 rad)  — matches D435 depth module                   -->
+    <!-- Resolution : 1280×720  — D435 max stereo resolution                       -->
+    <!-- Baseline : 0.05 m  — D435 IR baseline = 50 mm                             -->
+    <!-- Near clip : 0.1 m  — matches D435 min depth range                         -->
     <xacro:if value="$(arg stereo_camera_enabled)">
         <gazebo reference="stereo_camera">
             <sensor type="camera" name="right">
-                <update_rate>10.0</update_rate>
+                <update_rate>30.0</update_rate>
                 <always_on>true</always_on>
                 <ignition_frame_id>stereo_camera_optical</ignition_frame_id>
-                <pose>0 -0.12 0 0 0 0</pose>
+                <!-- right IR at -baseline/2 = -0.025 m from center -->
+                <pose>0 -0.025 0 0 0 0</pose>
                 <topic>stereo_camera/right/image_raw</topic>
                 <camera_info_topic>stereo_camera/right/camera_info</camera_info_topic>
-                <horizontal_fov>1.3962634</horizontal_fov>
+                <!-- D435 depth H-FOV = 87° = 1.5184 rad -->
+                <horizontal_fov>1.5184</horizontal_fov>
                 <image>
-                    <width>1024</width>
-                    <height>1024</height>
+                    <!-- D435 stereo resolution 1280×720 -->
+                    <width>1280</width>
+                    <height>720</height>
                     <format>R8G8B8</format>
                 </image>
                 <clip>
-                    <near>0.3</near>
-                    <far>20</far>
+                    <near>0.1</near>
+                    <far>10.0</far>
                 </clip>
             </sensor>
             <sensor type="camera" name="left">
                 <topic>stereo_camera/left/image_raw</topic>
-                <update_rate>10.0</update_rate>
+                <update_rate>30.0</update_rate>
                 <always_on>true</always_on>
                 <ignition_frame_id>stereo_camera_optical</ignition_frame_id>
                 <camera_info_topic>stereo_camera/left/camera_info</camera_info_topic>
-                <pose>0 0 0 0 0 0</pose>
-                <horizontal_fov>1.3962634</horizontal_fov>
+                <!-- left IR at +baseline/2 = +0.025 m from center -->
+                <pose>0 0.025 0 0 0 0</pose>
+                <horizontal_fov>1.5184</horizontal_fov>
                 <image>
-                    <width>1024</width>
-                    <height>1024</height>
+                    <width>1280</width>
+                    <height>720</height>
                     <format>R8G8B8</format>
                 </image>
                 <clip>
-                    <near>0.3</near>
-                    <far>20</far>
+                    <near>0.1</near>
+                    <far>10.0</far>
                 </clip>
             </sensor>
